File: Kicad/ch32v307_100/ch32v307_100.kicad_pcb (KiCad board)
At the start: 2 copper layers, 111.8 x 59.4 mm, 81 parts, among them J1 Conn_01x02, J10 USB_C_Receptacle_USB2.0, J2 Conn_02x10_Odd_Even, J3 Conn_02x10_Odd_Even, J4 Conn_01x04, J5 Conn_01x04, J6 Conn_01x02, J7 Conn_02x17_Odd_Even, J8 Conn_01x40, J9 Micro_SD_Card_Det, Q1 Q_NJFET_GSD, SW1 SW_RESET, SW2 SW_BOOT0, U1 AP2204RB-3.3, U2 AP2204RB-3.3, U3 CH32C307VCT6, U4 XPT2046TS, U5 74LS574, U6 74LS574, U7 CY7C1051DV33, U8 AP2204RB-3.3, Y1 32768 kHz, Y2 8 MHz

Commit message: Add files via upload
Parts:
- added R20: 10k, Resistor_SMD:R_0603_1608Metric, F.Cu at (53.3, 74.7)
Routing:
- net /+3.3V: track 371.7 -> 380.9 mm, vias 19 -> 21
- net Net-(J6-Pad1): track 5.01 -> 8.30 mm
- net /Y+: track 26.6 -> 28.3 mm
Other:
- board text added: "Rx1"
- board text added: "Tx1"

Commit message: Add files via upload
Connections:
- J8 pad 10: /RS(A0) -> /ADR21
- J8 pad 11: /WR(SCL) -> /LCD_WR
- J8 pad 12: /RD -> /ADR22
- J8 pad 9: /CS(CS) -> /LCD_CS
Routing:
- net /LCD_CS: track 41.9 -> 68.0 mm, vias 0 -> 3
- net /ADR22: track 50.2 -> 73.6 mm, vias 0 -> 3
- net /ADR21: track 47.5 -> 67.0 mm, vias 2 -> 5
- net /LCD_WR: track 67.2 -> 86.1 mm, vias 4 -> 6

Commit message: Add files via upload
Connections:
- J8 pad 15: /RESET -> /ADR20
Routing:
- net /ADR20: track 45.0 -> 70.2 mm, vias 1 -> 4
- net GND: track 622.2 -> 624.5 mm
- net /LCD_CS: track 68.0 -> 69.0 mm
- net /ADR21: track 67.0 -> 67.7 mm
- net /TFT_D5: track 55.7 -> 55.1 mm
