File: Kicad/ch32v307_100/ch32v307_100.sch (KiCad schematic (older format))
At the start: 76 parts, among them J1 Conn_01x02, J10 Conn_01x40, J2 Conn_02x10_Odd_Even, J3 Conn_01x04, J4 Conn_02x05_Odd_Even, J5 Conn_02x17_Odd_Even, J6 Micro_SD_Card_Det, J7 USB_C_Receptacle_USB2.0, J8 Conn_01x03, J9 Conn_01x04, SW1 SW_BOOT0, SW2 SW_BOOT0, U1 AMS1117-3.3, U2 AMS1117-3.3, U3 CH32C307VCT6, U4 74LS574, U5 74LS574, U6 CY7C1051DV33, U7 XPT2046TS, Y1 32768 kHz, Y2 8 MHz

Commit message: Add files via upload
Parts:
- removed J4: Conn_02x05_Odd_Even, symbol Connector_Generic:Conn_02x05_Odd_Even
- removed J8: Conn_01x03, symbol Connector_Generic:Conn_01x03
- removed R10, R11, R12, R13, R14, R15, R7, R8, R9: 470, symbol Device:R
- removed U1, U2: AMS1117-3.3, Package_TO_SOT_SMD:SOT-223-3_TabPin2, symbol Regulator_Linear:AMS1117-3.3
- added C28: 0.1, Capacitor_SMD:C_0603_1608Metric, symbol Device:C
- added C29, C30: 220.0uf, Capacitor_SMD:CP_Elec_6.3x5.4, symbol Device:CP
- added D2: LED, LED_SMD:LED_0805_2012Metric, symbol Device:LED
- added J2: Conn_02x10_Odd_Even, Connector_PinHeader_2.54mm:PinHeader_2x10_P2.54mm_Vertical, symbol Connector_Generic:Conn_02x10_Odd_Even
- added J6: Conn_01x02, Connector_PinHeader_2.54mm:PinHeader_1x02_P2.54mm_Vertical, symbol Connector_Generic:Conn_01x02
- added Q1: Q_NJFET_GSD, Package_TO_SOT_SMD:SC-59_Handsoldering, symbol Device:Q_NJFET_GSD
- added R18: 10k, Resistor_SMD:R_0603_1608Metric, symbol Device:R
- added R19: 10 0805, Resistor_SMD:R_0805_2012Metric, symbol Device:R
- added RN1, RN2: 470, Resistor_SMD:R_Array_Convex_4x0612, symbol Device:R_Pack04
- added U1, U2, U8: AP2204RB-3.3, Package_TO_SOT_SMD:SOT-89-3, symbol Regulator_Linear:AP2204RB-3.3
- BT1: footprint (none) -> my_battary:Battery_CR1225_SMD
- C1, C2, R1, R2, R3, R5, R6: footprint (none) -> Resistor_SMD:R_0603_1608Metric
- C10, C11, C12, C14, C15, C17, C18, C19, C20, C21, C23, C5, C6, C7, C8: footprint (none) -> Capacitor_SMD:C_0603_1608Metric
- C13, C22: footprint (none) -> Capacitor_THT:CP_Radial_D6.3mm_P2.50mm
- C16: value 100.0uf -> 220.0uf; footprint (none) -> Capacitor_SMD:CP_Elec_6.3x5.4
- C24: footprint (none) -> Capacitor_SMD:CP_Elec_5x5.4
- C25: renamed from C27; footprint (none) -> Capacitor_SMD:C_0603_1608Metric
- C26: renamed from C25; footprint (none) -> Capacitor_SMD:C_0603_1608Metric
- C27: renamed from C26; footprint (none) -> Capacitor_SMD:CP_Elec_4x5.4
- C3, C4: footprint (none) -> Capacitor_SMD:CP_Elec_4x5.4
- C9: footprint (none) -> Capacitor_SMD:C_0805_2012Metric
- D1: footprint (none) -> Diode_SMD:D_1210_3225Metric
- J1: footprint (none) -> Connector_PinHeader_2.54mm:PinHeader_1x02_P2.54mm_Vertical
- J10: renamed from J7; footprint (none) -> Connector_USB:USB_C_Receptacle_Palconn_UTC16-G
- J3: renamed from J2; footprint (none) -> Connector_PinHeader_2.54mm:PinHeader_2x10_P2.54mm_Vertical
- J4: renamed from J9; footprint (none) -> Connector_PinHeader_2.54mm:PinHeader_1x04_P2.54mm_Vertical
- J5: renamed from J3; footprint (none) -> Connector_PinHeader_2.54mm:PinHeader_1x04_P2.54mm_Vertical
- J7: renamed from J5; footprint (none) -> Connector_PinHeader_2.54mm:PinHeader_2x17_P2.54mm_Vertical
- J8: renamed from J10; footprint (none) -> Connector_FFC-FPC:Hirose_FH12-40S-0.5SH_1x40-1MP_P0.50mm_Horizontal
- J9: renamed from J6; footprint (none) -> my_sdcard:microSD__my_footprint
- R10: renamed from R20; footprint (none) -> Resistor_SMD:R_0603_1608Metric
- R11: renamed from R21; footprint (none) -> Resistor_SMD:R_0603_1608Metric
- R12: renamed from R22; footprint (none) -> Resistor_SMD:R_0603_1608Metric
- R13: renamed from R23; footprint (none) -> Resistor_SMD:R_0603_1608Metric
- R14: renamed from R24; footprint (none) -> Resistor_SMD:R_0603_1608Metric
- R15: renamed from R25; footprint (none) -> Resistor_SMD:R_0603_1608Metric
- R16: value 470 -> 1k; footprint (none) -> Resistor_SMD:R_0603_1608Metric
- R17: value 470 -> 10k; footprint (none) -> Resistor_SMD:R_0603_1608Metric
- R4: footprint (none) -> Resistor_SMD:R_0805_2012Metric
- R7: renamed from R26; footprint (none) -> Resistor_SMD:R_0603_1608Metric
- R8: renamed from R18; footprint (none) -> Resistor_SMD:R_0603_1608Metric
- R9: renamed from R19; footprint (none) -> Resistor_SMD:R_0603_1608Metric
- SW1: value SW_BOOT0 -> SW_RESET; footprint (none) -> my_push-buttons:SW_PUSH_6.0x3.2mm
- SW2: footprint (none) -> my_push-buttons:SW_PUSH_6.0x3.2mm
- U3: footprint (none) -> Package_QFP:LQFP-100_14x14mm_P0.5mm
- U4: renamed from U7; footprint Package_SO:TSSOP-14_4.4x5mm_P0.65mm -> Package_SO:TSSOP-16_4.4x5mm_P0.65mm
- U5: renamed from U4; footprint (none) -> Package_SO:SSOP-20_4.4x6.5mm_P0.65mm
- U6: renamed from U5; footprint (none) -> Package_SO:SSOP-20_4.4x6.5mm_P0.65mm
- U7: renamed from U6; footprint Package_SO:SOJ-44_10.16x28.58mm_P1.27mm -> Package_SO:TSOP-II-44_10.16x18.41mm_P0.8mm
- Y1: footprint (none) -> Crystal:Crystal_SMD_3215-2Pin_3.2x1.5mm
- Y2: footprint (none) -> Crystal:Crystal_SMD_3225-4Pin_3.2x2.5mm_HandSoldering
Connections:
- net IM1 is gone; now on net IM0: J8.39 (Pin_39)
- net IM2 is gone; now on net GND: J8.40 (Pin_40)
- net K2 is gone; now on net K1: J8.35 (Pin_35)
- net K3 is gone; now on net K1: J8.36 (Pin_36)
- net +3.3V: now also J9.4 (VDD), C30.1, D2.2 (A), J2.13 (Pin_13), J2.15 (Pin_15), U2.1 (VOUT); no longer D1.1 (K), J7.23 (Pin_23), J7.26 (Pin_26), J8.6 (Pin_6), J8.7 (Pin_7)
- net +5V: now also D1.1 (K), J2.16 (Pin_16), U1.3 (VIN), U2.3 (VIN), U8.3 (VIN)
- net ADR19: now also J2.12 (Pin_12)
- net AIN0: now also RN1.1 (R1.1), RN2.4 (R4.1); no longer R17.2
- net AIN1: now also RN1.2 (R2.1), RN2.3 (R3.1); no longer R16.2
- net AIN2: now also RN1.3 (R3.1), RN2.2 (R2.1)
- net AIN3: now also RN1.4 (R4.1), RN2.1 (R1.1)
- net AIN4: now also J2.11 (Pin_11)
- net FSMC_CLK: now also J2.14 (Pin_14)
- net GND: now also C28.1, C29.2, C30.2, J2.17 (Pin_17), J2.18 (Pin_18), J2.19 (Pin_19), J2.20 (Pin_20), Q1.2 (S), RN2.5 (R4.2), RN2.6 (R3.2), RN2.7 (R2.2), RN2.8 (R1.2), U1.2 (GND), U2.2 (GND), U8.2 (GND); no longer R17.1
- net IM0: now also R17.1
- net K1: now also R19.2
- net LCD_BKL: now also R18.1
- net SPI2_CLK: now also J2.4 (Pin_4)
- net SPI2_CS: now also J2.10 (Pin_10), J6.2 (Pin_2); no longer U4.15 (~CS)
- net SPI2_MISO: now also J2.8 (Pin_8)
- net SPI2_MOSI: now also J2.6 (Pin_6)
- net TFT_A: now also J7.23 (Pin_23), J7.26 (Pin_26), J8.6 (Pin_6), J8.7 (Pin_7), R17.2, C28.2, C29.1, U8.1 (VOUT)
- net URX4: now also J2.2 (Pin_2)
- net UTX4: now also J2.1 (Pin_1)
- net VDD_RAM: now also U1.1 (VOUT)
- net X+: now also J4.4 (Pin_4), U4.2 (XP)
- net X-: now also J4.2 (Pin_2), U4.4 (XN)
- net Y+: now also J4.3 (Pin_3), U4.3 (YP)
- net Y-: now also J4.1 (Pin_1), U4.5 (YN)
- net RS(SCL) renamed RS(A0)
- net WR(A0) renamed WR(SCL)
- new net: J6.1 (Pin_1), U4.15 (~CS)
- new net: J2.9 (Pin_9), RN1.5 (R4.2)
- new net: J2.7 (Pin_7), RN1.6 (R3.2)
- new net: J2.5 (Pin_5), RN1.7 (R2.2)
- new net: J2.3 (Pin_3), RN1.8 (R1.2)
- new net: Q1.1 (G), R18.2
- new net: Q1.3 (D), R19.1
- new net: D2.1 (K), R16.2
Other:
- moved on the sheet: C10, C11, C12, C13, C14, C15, C16, C17, C18, C19, C20, C21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

Commit message: Add files via upload
Parts:
- added R20: 10k, Resistor_SMD:R_0603_1608Metric, symbol Device:R
Connections:
- net +3.3V: now also R20.2
- net at J6.1 (Pin_1), U4.15 (~CS): now also R20.1
Changed lines of the file:
@@
 U 1 1 69211725
 P 6175 5075
-F 0 "R7" V 6125 5200 50  0000 L CNN
-F 1 "10k" V 6125 5350 50  0000 L CNN
+F 0 "R7" V 6125 4650 50  0000 L CNN
+F 1 "10k" V 6125 4825 50  0000 L CNN
 F 2 "Resistor_SMD:R_0603_1608Metric" V 6105 5075 50  0001 C CNN
 F 3 "~" H 6175 5075 50  0001 C CNN
@@
 $EndComp
 Wire Wire Line
-	6900 5750 6900 4700
+	6900 5750 6900 4975
 Wire Wire Line
 	6900 4700 6500 4700
@@
 Text Label 6925 7050 2    50   ~ 0
 FSMC_CLK
+$Comp
+L Device:R R20
+U 1 1 690B2FE2
+P 6175 4975
+F 0 "R20" V 6125 4550 50  0000 L CNN
+F 1 "10k" V 6125 4725 50  0000 L CNN
+F 2 "Resistor_SMD:R_0603_1608Metric" V 6105 4975 50  0001 C CNN
+F 3 "~" H 6175 4975 50  0001 C CNN
+	1    6175 4975
+	0    1    1    0
+$EndComp
+Wire Wire Line
+	6025 4975 5900 4975
+Wire Wire Line
+	5900 4975 5900 5075
+Connection ~ 6900 4975
+Wire Wire Line
+	6900 4975 6900 4700
+Wire Wire Line
+	6325 4975 6900 4975
 $EndSCHEMATC

Commit message: Add files via upload
Connections:
- net CS(CS) is gone; now on net LCD_CS: J8.9 (Pin_9)
- net RD is gone; now on net ADR22: J8.12 (Pin_12)
- net RS(A0) is gone; now on net ADR21: J8.10 (Pin_10)
- net WR(SCL) is gone; now on net LCD_WR: J8.11 (Pin_11)
Changed lines of the file:
@@
 FMARK
 Text Label 10275 5900 3    50   ~ 0
-CS(CS)
+LCD_CS
 Text Label 10175 5900 3    50   ~ 0
-RS(A0)
+LCD_RS
 Text Label 10075 5900 3    50   ~ 0
-WR(SCL)
+LCD_WR
 Text Label 9975 5900 3    50   ~ 0
-RD
+LCD_RD
 Text Label 10575 5900 3    50   ~ 0
 VDD_TFT

Commit message: Add files via upload
Connections:
- net RESET is gone; now on net ADR20: J8.15 (Pin_15)
Changed lines of the file:
@@
 SPI_SDO
 Text Label 9675 5900 3    50   ~ 0
-RESET
+LCD_RST
 Text Label 9575 5900 3    50   ~ 0
 GND
